File: kicad/plts-monitoring/plts-monitoring.kicad_sch (KiCad schematic)
At the start: 0 parts

Commit message: Add Micro SD Card footprint
Parts:
- added J1: Micro_SD_Card, Connector:J_SD_Card-micro_socket_A, symbol Connector:Micro_SD_Card
- added U1: ATmega328P-A, Package_QFP:TQFP-32_7x7mm_P0.8mm, symbol MCU_Microchip_ATmega:ATmega328P-A
- added U2: DS3232M, Package_SO:SOIC-8_3.9x4.9mm_P1.27mm, symbol Timer_RTC:DS3232M
Connections:
- new net: U1.21 (GND), U1.3 (GND), U1.5 (GND)
- new net: U1.4 (VCC), U1.6 (VCC)
Changed lines of the file:
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@@
 (kicad_sch (version 20230121) (generator eeschema)
-  (paper "A4")
+  (paper "A3")
   (title_block
     (title "plts-monitoring-board")
@@
     (comment 2 "Author: Ahmad Qodri")
   )
+  (symbol (lib_id "MCU_Microchip_ATmega:ATmega328P-A") (at 142.24 76.2 0) (unit 1)
+    (in_bom yes) (on_board yes) (dnp no) (fields_autoplaced)
+    (property "Reference" "U1" (at 144.4341 114.3 0)
+      (effects (font (size 1.27 1.27)) (justify left))
+    )
+    (property "Value" "ATmega328P-A" (at 144.4341 116.84 0)
+      (effects (font (size 1.27 1.27)) (justify left))
+    )
+    (property "Footprint" "Package_QFP:TQFP-32_7x7mm_P0.8mm" (at 142.24 76.2 0)
+      (effects (font (size 1.27 1.27) italic) hide)
+    )
+    (property "Datasheet" "http://ww1.microchip.com/downloads/en/DeviceDoc/ATmega328_P%20AVR%20MCU%20with%20picoPower%20Technology%20Data%20Sheet%2040001984A.pdf" (at 142.24 76.2 0)
+      (effects (font (size 1.27 1.27)) hide)
+    )
+    (pin "4")
+    (pin "32")
+    (pin "31")
+    (pin "24")
+    (pin "2")
+    (pin "13")
+    (pin "17")
+    (pin "26")
+    (pin "28")
+    (pin "12")
+    (pin "11")
+    (pin "3")
+    (pin "5")
+    (pin "15")
+    (pin "20")
+    (pin "25")
+    (pin "6")
+    (pin "30")
+    (pin "1")
+    (pin "29")
+    (pin "14")
+    (pin "19")
+    (pin "18")
+    (pin "21")
+    (pin "27")
+    (pin "8")
+    (pin "9")
+    (pin "23")
+    (pin "22")
+    (pin "16")
+    (pin "7")
+    (pin "10")
+    (instances
+      (project "plts-monitoring"
+        (path "/766d1dbc-8b07-4f68-b453-e8f5a8eb62fa"
+          (reference "U1") (unit 1)
+        )
+      )
+    )
+  )
+  (symbol (lib_id "Timer_RTC:DS3232M") (at 203.2 52.07 0) (unit 1)
+    (in_bom yes) (on_board yes) (dnp no) (fields_autoplaced)
+    (property "Reference" "U2" (at 205.3941 62.23 0)
+      (effects (font (size 1.27 1.27)) (justify left))
+    )
+    (property "Value" "DS3232M" (at 205.3941 64.77 0)
+      (effects (font (size 1.27 1.27)) (justify left))
+    )
+    (property "Footprint" "Package_SO:SOIC-8_3.9x4.9mm_P1.27mm" (at 204.47 64.77 0)
+      (effects (font (size 1.27 1.27)) hide)
+    )
+    (property "Datasheet" "http://datasheets.maximintegrated.com/en/ds/DS3232M.pdf" (at 210.058 48.26 0)
+      (effects (font (size 1.27 1.27)) hide)
+    )
+    (pin "5")
+    (pin "1")
+    (pin "2")
+    (pin "6")
+    (pin "7")
+    (pin "4")
+    (pin "3")
+    (pin "8")
+    (instances
+      (project "plts-monitoring"
+        (path "/766d1dbc-8b07-4f68-b453-e8f5a8eb62fa"
+          (reference "U2") (unit 1)
+        )
+      )
+    )
+  )
+  (symbol (lib_id "Connector:Micro_SD_Card") (at 224.79 104.14 0) (unit 1)
+    (in_bom yes) (on_board yes) (dnp no)
+    (property "Reference" "J1" (at 225.425 85.09 0)
+      (effects (font (size 1.27 1.27)))
+    )
+    (property "Value" "Micro_SD_Card" (at 225.425 87.63 0)
+      (effects (font (size 1.27 1.27)))
+    )
+    (property "Footprint" "Connector:J_SD_Card-micro_socket_A" (at 223.52 123.19 0)
+      (effects (font (size 1.27 1.27)))
+    )
+    (property "Datasheet" "http://katalog.we-online.de/em/datasheet/693072010801.pdf" (at 224.79 104.14 0)
+      (effects (font (size 1.27 1.27)) hide)
+    )
+    (pin "2")
+    (pin "1")
+    (pin "3")
+    (pin "4")
+    (pin "8")
+    (pin "5")
+    (pin "6")
+    (pin "7")
+    (pin "9")
+    (instances
+      (project "plts-monitoring"
+        (path "/766d1dbc-8b07-4f68-b453-e8f5a8eb62fa"
+          (reference "J1") (unit 1)
+        )
+      )
+    )
+  )
   (sheet_instances

Commit message: Update KiCad schematic
Parts:
- added BT1: Battery_Cell, Battery:BatteryHolder_Keystone_3000_1x12mm, symbol Device:Battery_Cell
- added C1, C2: 22p, Capacitor_SMD:C_0805_2012Metric, symbol Device:C
- added C10, C11: 1nF, Capacitor_Tantalum_SMD:CP_EIA-1608-10_AVX-L, symbol Device:C
- added C12, C15, C16: 100pF, Capacitor_Tantalum_SMD:CP_EIA-1608-10_AVX-L, symbol Device:C
- added C13, C14: 100nF, Capacitor_Tantalum_SMD:CP_EIA-1608-10_AVX-L, symbol Device:C
- added C3: 100uF, Capacitor_SMD:CP_Elec_5x5.7, symbol Device:C
- added C4: 1000uF, Capacitor_SMD:CP_Elec_5x5.7, symbol Device:C
- added C5: 10uF, Capacitor_Tantalum_SMD:CP_EIA-2012-12_Kemet-R, symbol Device:C
- added C6: 22uF, Capacitor_Tantalum_SMD:CP_EIA-2012-12_Kemet-R, symbol Device:C
- added C7: 0.1uF, Capacitor_Tantalum_SMD:CP_EIA-2012-12_Kemet-R, symbol Device:C
- added C8, C9: 0.1uF, Capacitor_Tantalum_SMD:CP_EIA-1608-10_AVX-L, symbol Device:C
- added D1: 1N5822, Diode_THT:D_DO-201AD_P15.24mm_Horizontal, symbol Diode:1N5822
- added D2: LED, symbol Device:LED
- added D3: 1N4448W, Diode_SMD:D_SOD-123, symbol Diode:1N4448W
- added DS1: WC1602A, Display:WC1602A, symbol Display_Character:WC1602A
- added J2, J4: 7-40VDC, TerminalBlock_Phoenix:TerminalBlock_Phoenix_MKDS-1,5-2-5.08_1x02_P5.08mm_Horizontal, symbol Connector:Screw_Terminal_01x02
- added J3: AVR-ISP-10, symbol Connector:AVR-ISP-10
- added L1: 100uH, Inductor_SMD:L_Bourns_SRR1210A, symbol Device:L
- added R1, R10, R12, R13, R14, R15, R16, R2, R4, R5, R6, R7, R8: 10k, Resistor_SMD:R_0805_2012Metric, symbol Device:R
- added R11: 1k, Resistor_SMD:R_0805_2012Metric, symbol Device:R
- added R3: 330, Resistor_SMD:R_0805_2012Metric, symbol Device:R
- added R9: 2k, Resistor_SMD:R_0805_2012Metric, symbol Device:R
- added RV1: R_Potentiometer_US, Potentiometer_SMD:Potentiometer_Bourns_3224X_Vertical, symbol Device:R_Potentiometer_US
- added SW2: SW_Push_Dual, Button_Switch_THT:SW_PUSH_6mm_H4.3mm, symbol Switch:SW_Push_Dual
- added U3: ACS712xLCTR-30A, Package_SO:SOIC-8_3.9x4.9mm_P1.27mm, symbol Sensor_Current:ACS712xLCTR-30A
- added U4: ACPL-C87B, Package_SO:SSO-8_6.8x5.9mm_P1.27mm_Clearance8mm, symbol Isolator_Analog:ACPL-C87B
- added U5: OPA2376xxD, Package_SO:TSSOP-8_3x3mm_P0.65mm, symbol Amplifier_Operational:OPA2376xxD
- added U6: AMS1117-3.3, Package_TO_SOT_SMD:SOT-223-3_TabPin2, symbol Regulator_Linear:AMS1117-3.3
- added U7: LM2576HVS-5, Package_TO_SOT_SMD:TO-263-5_TabPin3, symbol Regulator_Switching:LM2576HVS-5
- added Y1: 16MHz, Crystal:Crystal_SMD_2012-2Pin_2.0x1.2mm, symbol Device:Crystal
- J1: footprint Connector:J_SD_Card-micro_socket_A -> Connector_Card:microSD_HC_Hirose_DM3D-SF
Connections:
- net PD3/3: now reaches U1.1 (PD3)
- net PD3/3: now also DS1.6 (E)
- net PD6/6: now reaches U1.10 (PD6)
- net PD6/6: now also DS1.13 (D6)
- net PD7/7: now reaches U1.11 (PD7)
- net PD7/7: now also DS1.14 (D7)
- net PB0/8: now reaches U1.12 (PB0)
- net PB1/9: now reaches U1.13 (PB1)
- net PB2/10: now reaches U1.14 (PB2)
- net PB2/10: now also J1.2 (DAT3/CD), R1.2
- net PB3/11/MOSI: now reaches U1.15 (PB3)
- net PB3/11/MOSI: now also J1.3 (CMD), J3.1 (MOSI)
- net PB4/12/MISO: now reaches U1.16 (PB4)
- net PB4/12/MISO: now also J1.7 (DAT0), J3.9 (MISO), R6.2
- net PB5/13/SCK: now reaches U1.17 (PB5)
- net PB5/13/SCK: now also J1.5 (CLK), J3.7 (SCK)
- net +5V: now reaches U1.18 (AVCC)
- net +5V: now also U1.20 (AREF), U1.4 (VCC), U1.6 (VCC), U2.2 (VCC), C14.1, C4.1, C5.1, C9.2, D2.2 (A), DS1.15 (LED(+)), DS1.2 (VDD), J3.2 (VCC), L1.2, R2.1, R4.1, R5.1, RV1.1, U4.8 (VDD2), U6.3 (VI), U7.4 (FB)
- net ADC/A6: now reaches U1.19 (ADC6)
- net ADC/A6: now also U1.22 (ADC7)
- net PD4/4: now reaches U1.2 (PD4)
- net PD4/4: now also DS1.11 (D4)
- net GND: now reaches U1.21 (GND), U1.3 (GND), U1.5 (GND)
- net GND: now also J1.6 (VSS), J1.9 (SHIELD), U2.5 (GND), BT1.2 (-), C1.2, C10.2, C11.2, C12.2, C13.2, C14.2, C15.1, C2.1, C3.2, C4.2, C5.2, C6.2, C7.2, C8.2, C9.1, D1.2 (A), DS1.16 (LED(-)), DS1.5 (R/W), J2.1 (Pin_1), J3.10 (GND), J3.4 (GND), J3.6 (GND), J3.8 (GND), R10.1, R11.2, R15.1, R3.2, RV1.3, SW2.2, SW2.4, U3.5 (GND), U4.3 (IN-), U4.4 (GND1), U4.5 (GND2), U6.1 (GND), U7.3 (GND), U7.5 (~{ON}/OFF)
- net PC0/A0/14: now reaches U1.23 (PC0)
- net PC0/A0/14: now also C11.1, D3.1 (K)
- net PC1/A1/15: now reaches U1.24 (PC1)
- net PC1/A1/15: now also C16.2, R16.1, U5.1
- net PC2/A2/16: now reaches U1.25 (PC2)
- net PC3/A3/17: now reaches U1.26 (PC3)
- net PC4/A4/18/SDA: now reaches U1.27 (PC4)
- net PC4/A4/18/SDA: now also U2.7 (SDA), R5.2
- net PC4/A5/19/SCL: now reaches U1.28 (PC5)
- net PC4/A5/19/SCL: now also U2.8 (SCL), R4.2
- net RST: now reaches U1.29 (~{RESET}/PC6)
- net RST: now also U2.4 (~{RST}), J3.5 (~{RST}), R2.2, SW2.1, SW2.3
- net PD0/0/RXD: now reaches U1.30 (PD0)
- net PD0/1/TXD: now reaches U1.31 (PD1)
- net PD2/2: now reaches U1.32 (PD2)
- net PD2/2: now also DS1.4 (RS)
- net XTAL1: now reaches U1.7 (XTAL1/PB6)
- net XTAL1: now also C1.1, Y1.1
- net XTAL2: now reaches U1.8 (XTAL2/PB7)
- net XTAL2: now also C2.2, Y1.2
- net PD5/5: now reaches U1.9 (PD5)
- net PD5/5: now also DS1.12 (D5)
- net at U2.6 (VBAT): now also BT1.1 (+), C8.1
- net at J1.1 (DAT2): now also R8.2
- net +3.3V: now reaches J1.4 (VDD)
- net +3.3V: now also C6.1, C7.1, R1.1, R6.1, R7.1, R8.1, U6.2 (VO)
- net at J1.8 (DAT1): now also R7.2
- new net: C16.1, R14.2, R16.2, U5.2 (-)
- new net: C15.2, R13.1, R15.2, U5.3 (+)
- new net: D2.1 (K), R3.1
- new net: D3.2 (A), R10.2, R9.1
- new net: R9.2, U3.7 (VIOUT)
- new net: J4.1 (Pin_1), U3.3 (IP-), U3.4 (IP-)
- new net: C10.1, U3.6 (FILTER)
- new net: DS1.3 (VO), RV1.2
- new net: D1.1 (K), L1.1, U7.2 (OUT)
- new net: C12.1, R11.1, R12.2, U4.2 (IN)
- new net: R14.1, U4.6 (OUT-)
- new net: R13.2, U4.7 (OUT+)
- new net +BATT: C3.1, J2.2 (Pin_2), U7.1 (VIN)
- new net V_SolarPanel: C13.1, J4.2 (Pin_2), R12.1, U3.1 (IP+), U3.2 (IP+), U4.1 (VDD1)
Other:
- note added: "AVR Minimum System"
- note added: "Current Sensor"
- note added: "DC SUPPLY"
- note added: "LCD 16x02"
- note added: "Micro SD Card Interfacing"
- note added: "RTC Module"
- note added: "Voltage Sensor"
- moved on the sheet: J1, U1, U2

Commit message: Update schematic to pass ERC and some footprints
Parts:
- removed SW2: SW_Push_Dual, Button_Switch_THT:SW_PUSH_6mm_H4.3mm, symbol Switch:SW_Push_Dual
- added SW1: SW_Push, Button_Switch_THT:SW_PUSH_6mm_H4.3mm, symbol Switch:SW_Push
- added unit 3 of U7
- D2: footprint (none) -> LED_SMD:LED_0805_2012Metric
- J2: renamed from J3; footprint (none) -> Connector_IDC:IDC-Header_2x05_P2.54mm_Vertical
- L1: footprint Inductor_SMD:L_Bourns_SRR1210A -> Inductor_SMD:L_Bourns_SRP7028A_7.3x6.6mm
- renumbered C8 to C1, C13 to C10, C10 to C11, C11 to C12, C14 to C13, C15 to C14, C16 to C15, C7 to C16, C3 to C2, C4 to C3, C5 to C4, C1 to C5, C2 to C6, C6 to C7, C9 to C8, C12 to C9, J2 to J1, J4 to J3, J1 to J4, R2 to R1, R14 to R10, R15 to R11, R16 to R12, R8 to R13, R7 to R14, R6 to R15, R1 to R16, R3 to R2, R4 to R3, R5 to R4, R12 to R5, R11 to R6, R9 to R7, R10 to R8, R13 to R9, U7 to U2, U2 to U3, U6 to U4, U3 to U5, U4 to U6, U5 to U7
Connections:
- net +5V: now also U5.8 (VCC), U7.8 (V+)
- net GND: now also DS1.1 (VSS), SW1.2, U7.4 (V-)
- net RST: now also SW1.1
